Commit message: added more support for the ouster lidar

File: data/hail_bopp.urdf (robot description, URDF)
Before this commit: robot voltron, 10 links, 9 joints
Joints:
- added joint lidar_ouster_joint: type fixed, parent base_link, child os_lidar, origin xyz=0.0 0.68 1.8 rpy=0.15 0.2 0.55

Commit message: edits while testing ouster lidar

File: data/hail_bopp.urdf (robot description, URDF)
Before this commit: robot voltron, 10 links, 10 joints
Links:
- added link lidar_ouster
Joints:
- joint lidar_ouster_joint: child os_lidar -> lidar_ouster

Commit message: changes to get ouster lidar working

File: data/hail_bopp.urdf (robot description, URDF)
Before this commit: robot voltron, 11 links, 10 joints
Links:
- removed link lidar_ouster
- added link os_sensor
Joints:
- joint lidar_ouster_joint: child lidar_ouster -> os_sensor

Commit message: more fixes for the new lidar

File: data/hail_bopp.urdf (robot description, URDF)
Before this commit: robot voltron, 11 links, 10 joints
Joints:
- joint lidar_ouster_joint: origin xyz=0.0 0.68 1.8 rpy=0.15 0.2 0.55 -> xyz=0.0 0.58 1.8 rpy=0.0 0.2 0.0

Commit message: Ouster lidar transforms and destIP set

File: data/hail_bopp.urdf (robot description, URDF)
Before this commit: robot voltron, 11 links, 10 joints
Joints:
- joint lidar_ouster_joint: origin xyz=0.0 0.58 1.8 rpy=0.0 0.2 0.0 -> xyz=-1.32 0.0 1.8 rpy=0.0 0.0 0.0
